File: pcb/DmxAnalogLed.brd (EAGLE design)
At the start: 62 parts, among them IC2 7805TV, J1 RS485, J2 POWER_JACKPTH, J3 RS485, Q1 16MHz 10ppm, U1 ARDUINO_LEONARDO-REV3B_SMARTP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, U2 SN75176ASOIC, X1 USBPTH

Commit message: Update component values on PCB
Parts:
- JP4: value (none) -> DNP
- R1: value 180 -> 180 DNP
- R8: value 330 -> 470
Changed lines of the file:
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@@
 <elements>
 <element name="U2" library="reprap" package="SO08" value="SN75176ASOIC" x="66.5" y="24.5" smashed="yes" rot="R180"/>
-<element name="R1" library="SparkFun" package="0805" value="180" x="66.75" y="19.25" smashed="yes"/>
+<element name="R1" library="SparkFun" package="0805" value="180 DNP" x="66.75" y="19.25" smashed="yes"/>
 <element name="R2" library="SparkFun" package="0805" value="10k" x="66.25" y="30.25" smashed="yes" rot="R180"/>
-<element name="R8" library="SparkFun" package="0805" value="330" x="40.5" y="26.5" smashed="yes" rot="R180"/>
+<element name="R8" library="SparkFun" package="0805" value="470" x="40.5" y="26.5" smashed="yes" rot="R180"/>
 <element name="C7" library="SparkFun" package="0805" value="100nF" x="70.25" y="19.25" smashed="yes" rot="R180"/>
 <element name="J1" library="con-amp" package="520426-4" value="RS485" x="56" y="6.5" smashed="yes">
@@
 <attribute name="VALUE" x="42.77" y="69.48" size="0.4064" layer="27" rot="R180"/>
 </element>
-<element name="JP4" library="SparkFun" package="SCREWTERMINAL-3.5MM-4" value="" x="4.25" y="21.75" smashed="yes" rot="R270">
+<element name="JP4" library="SparkFun" package="SCREWTERMINAL-3.5MM-4" value="DNP" x="4.25" y="21.75" smashed="yes" rot="R270">
 <attribute name="VALUE" x="5.52" y="23.02" size="0.4064" layer="27" rot="R270"/>
 </element>
@@
 </signal>
 </signals>
-<errors>
-</errors>
 </board>
 </drawing>

Commit message: Get RevB ready
Parts:
- removed C18, C19, C20, C21: ?uF, SparkFun:1210
- removed JP4: DNP, SparkFun:SCREWTERMINAL-3.5MM-4
- added C22: .1uF, SparkFun:0805
- added C23, C24, C25, C26: (no value), SparkFun:PANASONIC_E
- C3: value 10uF -> .1uF
- C5, C6: value 100nF -> .1uF
- IC2: value 7805TV -> 7805DT; device linear:TO220V -> linear:TO252
- moved C10 24.1 mm to (57.0, 25.2), turned to 270 degrees
- moved C17 22.8 mm to (57.0, 25.2), turned to 90 degrees
- moved U$11 20.2 mm to (12.8, 44.0)
- moved IC2 17.9 mm to (13.8, 24.2), turned to 90 degrees
- moved C13 16.3 mm to (18.5, 17.2), turned to 270 degrees
- moved R12 14.4 mm to (59.8, 35.5)
- moved C11 14.1 mm to (18.5, 17.2), turned to 90 degrees
- moved U$12 13.2 mm to (62.5, 29.8)
- moved C7 11.2 mm to (59.5, 22.2), turned to 270 degrees
- moved C9 10.4 mm to (57.0, 35.5), turned to 90 degrees
- moved R2 10.3 mm to (71.8, 21.5), turned to 0 degrees
- moved U$10 9.33 mm to (53.5, 36.2), turned to 270 degrees
- moved C16 8.55 mm to (57.0, 35.5), turned to 270 degrees
- moved R1 6.26 mm to (61.2, 22.2), turned to 270 degrees
- moved C14 4.96 mm to (22.5, 30.2), turned to 90 degrees
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Connections:
- removed net V_PWM: C11.2, C13.1, C18.1, C19.1, C20.1, C21.1, IC2.1, J2.PWR, JP2.1, JP2.3, JP2.5, JP2.7, JP3.1, JP3.3, JP3.5, JP3.7, JP4.1, JP4.2
- new net V_IN: C11.2, C13.1, C23.+, C24.+, C25.+, C26.+, IC2.1, J2.PWR, JP2.1, JP2.3, JP2.5, JP2.7, JP3.1, JP3.3, JP3.5, JP3.7
- net GND: now also C22.1, C23.-, C24.-, C25.-, C26.-, IC2.3; no longer C18.2, C19.2, C20.2, C21.2, IC2.2, JP4.3, JP4.4
- net VCC: now also C22.2, IC2.2; no longer IC2.3
Routing:
- net GND: track 414.1 -> 83.9 mm, vias 17 -> 46
- net V_PWM: track 230.7 -> 0.00 mm, vias 4 -> 0
- net GND_ISO: track 87.6 -> 31.7 mm, vias 2 -> 18
- net PWM0: track 76.7 -> 99.5 mm
- net VCC: track 149.7 -> 132.7 mm, vias 3 -> 2
- net V_IN: track 0.00 -> 14.5 mm, vias 0 -> 20
- net 5V_ISO: track 37.5 -> 24.6 mm, vias 1 -> 0
- net RX: track 53.2 -> 44.1 mm
- net RS485A: track 31.5 -> 36.5 mm
- net N$14: track 11.4 -> 7.15 mm
- net PWM7: track 48.3 -> 52.1 mm
- net RS485B: track 24.9 -> 28.6 mm
- net PWM5: track 32.3 -> 35.3 mm, vias 0 -> 2
- net N$8: track 25.4 -> 28.3 mm, vias 0 -> 1
- net PWM6: track 42.6 -> 44.8 mm
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- added copper zone on layer 1, net GND
- added copper zone on layer 16, net GND
- added copper zone on layer 1, net GND_ISO
- added copper zone on layer 16, net GND_ISO
- added copper zone on layer 1, net V_IN
- added copper zone on layer 16, net V_IN
Other:
- board text added: "RevB 3/15"
- board text added: "keep it locked"
- board text removed: "RevA 3/13"

Commit message: RevB candidate; fixes ground plane, isolation, regulator placement, silk.
Parts:
- removed U$11: (no value), SparkFun:OSHW-LOGO-L
- added U$13: (no value), blinkiverse:OSHW-LOGO-L
- C15: value ?uF -> 1uF
Routing:
- net V_IN: vias 20 -> 15

Commit message: Make the software faster.
Parts:
- C12, C14, C22, C3, C5, C6: value .1uF -> 100nF
Changed lines of the file:
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@@
 <element name="R5" library="SparkFun" package="0805" value="22" x="30.4" y="14.25" smashed="yes" rot="R90"/>
 <element name="R6" library="SparkFun" package="0805" value="22" x="28.65" y="14.25" smashed="yes" rot="R90"/>
-<element name="C3" library="SparkFun" package="0805" value=".1uF" x="26.75" y="18.5" smashed="yes"/>
-<element name="C5" library="SparkFun" package="0805" value=".1uF" x="26.75" y="24.75" smashed="yes"/>
-<element name="C6" library="SparkFun" package="0805" value=".1uF" x="39.6" y="18" smashed="yes" rot="R90"/>
+<element name="C3" library="SparkFun" package="0805" value="100nF" x="26.75" y="18.5" smashed="yes"/>
+<element name="C5" library="SparkFun" package="0805" value="100nF" x="26.75" y="24.75" smashed="yes"/>
+<element name="C6" library="SparkFun" package="0805" value="100nF" x="39.6" y="18" smashed="yes" rot="R90"/>
 <element name="Q1" library="blinkyboard" package="XS3225" value="16MHz 10ppm" x="40.5" y="21.75" smashed="yes" rot="R270"/>
 <element name="C4" library="SparkFun" package="0805" value="1uF" x="32.5" y="14.25" smashed="yes" rot="R90">
@@
 <attribute name="VALUE" x="19.897" y="16.234" size="0.4064" layer="27" rot="R90"/>
 </element>
-<element name="C12" library="SparkFun" package="0805" value=".1uF" x="22.5" y="30.25" smashed="yes" rot="R270">
+<element name="C12" library="SparkFun" package="0805" value="100nF" x="22.5" y="30.25" smashed="yes" rot="R270">
 <attribute name="VALUE" x="21.103" y="31.266" size="0.4064" layer="27" rot="R270"/>
 </element>
@@
 <attribute name="VALUE" x="17.8" y="18.15" size="0.4064" layer="27" rot="R270"/>
 </element>
-<element name="C14" library="SparkFun" package="1210" value=".1uF" x="22.5" y="30.25" smashed="yes" rot="R90">
+<element name="C14" library="SparkFun" package="1210" value="100nF" x="22.5" y="30.25" smashed="yes" rot="R90">
 <attribute name="VALUE" x="23.2" y="29.35" size="0.4064" layer="27" rot="R90"/>
 </element>
@@
 <attribute name="VALUE" x="16.29" y="29.33" size="1.27" layer="27" rot="R180"/>
 </element>
-<element name="C22" library="SparkFun" package="0805" value=".1uF" x="36.75" y="27.75" rot="R270"/>
+<element name="C22" library="SparkFun" package="0805" value="100nF" x="36.75" y="27.75" rot="R270"/>
 <element name="C23" library="SparkFun" package="PANASONIC_E" value="" x="45.75" y="54.75" smashed="yes" rot="R90">
 <attribute name="VALUE" x="48.29" y="53.48" size="0.4064" layer="27" rot="R90"/>
