File: pcb/DmxAnalogLed.brd (EAGLE design)
At the start: 62 parts, among them IC2 7805DT, J1 RS485, J2 POWER_JACKPTH, J3 RS485, Q1 16MHz 10ppm, U1 ARDUINO_LEONARDO-REV3B_SMARTP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, U2 SN75176ASOIC, X1 USBPTH

Commit message: Change library name, too
Parts:
- U$1, U$3, U$4, U$5, U$6, U$7, U$8, U$9: device blinkiverse:TO252 -> blinkinlabs:TO252
- U$10: device blinkiverse:IB_XLS-1W -> blinkinlabs:IB_XLS-1W
- U$13: device blinkiverse:OSHW-LOGO-L -> blinkinlabs:OSHW-LOGO-L
- U1: device blinkiverse:ARDUINO_LEONARDO-REV3B_SMARTPRJ_QFN44ML7X7 -> blinkinlabs:ARDUINO_LEONARDO-REV3B_SMARTPRJ_QFN44ML7X7
Changed lines of the file:
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@@
 </element>
 <element name="U$2" library="sonos_library" package="2X3HEADER" value="2X3HEADER" x="41.75" y="11.75"/>
-<element name="U1" library="blinkiverse" package="ARDUINO_LEONARDO-REV3B_SMARTPRJ_QFN44ML7X7" value="ARDUINO_LEONARDO-REV3B_SMARTPRJ_ATMEGA32U4-XUMU" x="32.5" y="21.9" smashed="yes" rot="R90"/>
+<element name="U1" library="blinkinlabs" package="ARDUINO_LEONARDO-REV3B_SMARTPRJ_QFN44ML7X7" value="ARDUINO_LEONARDO-REV3B_SMARTPRJ_ATMEGA32U4-XUMU" x="32.5" y="21.9" smashed="yes" rot="R90"/>
 <element name="C1" library="SparkFun" package="0805" value="16pf" x="41.25" y="18" smashed="yes" rot="R90"/>
 <element name="C2" library="SparkFun" package="0805" value="16pf" x="40.5" y="24.75" smashed="yes" rot="R180"/>
@@
 <attribute name="VALUE" x="83.152" y="1.674" size="1.778" layer="27" rot="R90"/>
 </element>
-<element name="U$1" library="blinkiverse" package="TO252" value="N_MOSFET" x="74.5" y="59.75"/>
-<element name="U$3" library="blinkiverse" package="TO252" value="N_MOSFET" x="67.5" y="59.75"/>
-<element name="U$4" library="blinkiverse" package="TO252" value="N_MOSFET" x="60.5" y="59.75"/>
-<element name="U$5" library="blinkiverse" package="TO252" value="N_MOSFET" x="53.5" y="59.75"/>
-<element name="U$6" library="blinkiverse" package="TO252" value="N_MOSFET" x="38" y="59.75"/>
-<element name="U$7" library="blinkiverse" package="TO252" value="N_MOSFET" x="31" y="59.75"/>
-<element name="U$8" library="blinkiverse" package="TO252" value="N_MOSFET" x="24" y="59.75"/>
-<element name="U$9" library="blinkiverse" package="TO252" value="N_MOSFET" x="17" y="59.75"/>
+<element name="U$1" library="blinkinlabs" package="TO252" value="N_MOSFET" x="74.5" y="59.75"/>
+<element name="U$3" library="blinkinlabs" package="TO252" value="N_MOSFET" x="67.5" y="59.75"/>
+<element name="U$4" library="blinkinlabs" package="TO252" value="N_MOSFET" x="60.5" y="59.75"/>
+<element name="U$5" library="blinkinlabs" package="TO252" value="N_MOSFET" x="53.5" y="59.75"/>
+<element name="U$6" library="blinkinlabs" package="TO252" value="N_MOSFET" x="38" y="59.75"/>
+<element name="U$7" library="blinkinlabs" package="TO252" value="N_MOSFET" x="31" y="59.75"/>
+<element name="U$8" library="blinkinlabs" package="TO252" value="N_MOSFET" x="24" y="59.75"/>
+<element name="U$9" library="blinkinlabs" package="TO252" value="N_MOSFET" x="17" y="59.75"/>
 <element name="JP2" library="SparkFun" package="SCREWTERMINAL-3.5MM-8" value="" x="78" y="70.75" smashed="yes" rot="R180">
 <attribute name="VALUE" x="79.27" y="69.48" size="0.4064" layer="27" rot="R180"/>
@@
 <attribute name="VALUE" x="42.77" y="69.48" size="0.4064" layer="27" rot="R180"/>
 </element>
-<element name="U$10" library="blinkiverse" package="IB_XLS-1W" value="DC_DC_ISOLATED_0505" x="53.5" y="36.25" rot="R270"/>
+<element name="U$10" library="blinkinlabs" package="IB_XLS-1W" value="DC_DC_ISOLATED_0505" x="53.5" y="36.25" rot="R270"/>
 <element name="C9" library="SparkFun" package="0805" value="4.7uF" x="57" y="35.5" smashed="yes" rot="R90">
 <attribute name="VALUE" x="58.397" y="34.484" size="0.4064" layer="27" rot="R90"/>
@@
 <attribute name="VALUE" x="6.98" y="12.96" size="0.4064" layer="27"/>
 </element>
-<element name="U$13" library="blinkiverse" package="OSHW-LOGO-L" value="" x="12.75" y="44.25"/>
+<element name="U$13" library="blinkinlabs" package="OSHW-LOGO-L" value="" x="12.75" y="44.25"/>
 </elements>
 <signals>
